Commit message: fix some files

File: tripod_calibration_test/tripod_calib_test_description/urdf/tripod_rgb_rgb.gazebo.xacro (robot description, xacro)
@@ -1,17 +1,6 @@
 <?xml version="1.0"?>
 <robot xmlns:xacro="http://ros.org/wiki/xacro">
-<!-- add sensor camera RIGHT part -->
+  <!-- add sensor camera RIGHT part -->
   <xacro:macro name="sim_3dsensor" params="prefix">
-    <gazebo reference="${prefix}_depth_frame">
-      <sensor type="depth" name="camera">
-        <always_on>true</always_on>
-        <update_rate>20.0</update_rate>
-        <camera>
-          <horizontal_fov>${60.0*pi/180.0}</horizontal_fov>
-          <image>
-            <format>B8G8R8</format>
-            <width>640</width>
-            <height>480</height>
-          </image>  <xacro:macro name="sim_3dsensor" params="prefix">
     <gazebo reference="${prefix}_depth_frame">
       <sensor type="depth" name="camera">
@@ -51,44 +40,7 @@
     </gazebo>
   </xacro:macro>
-          <clip>
-            <near>0.10</near>
-            <far>8.0</far>
-          </clip>
-        </camera>
-        <plugin name="${prefix}_camera_controller" filename="libgazebo_ros_openni_kinect.so">
-          <cameraName>${prefix}</cameraName>
-          <alwaysOn>true</alwaysOn>
-          <updateRate>10</updateRate>
-          <imageTopicName>rgb/image_raw</imageTopicName>
-          <depthImageTopicName>depth/image_raw</depthImageTopicName>
-          <pointCloudTopicName>depth/points</pointCloudTopicName>
-          <cameraInfoTopicName>rgb/camera_info</cameraInfoTopicName>
-          <depthImageCameraInfoTopicName>depth/camera_info</depthImageCameraInfoTopicName>
-          <frameName>${prefix}_depth_optical_frame</frameName>
-          <baseline>0.1</baseline>
-          <distortion_k1>0.0</distortion_k1>
-          <distortion_k2>0.0</distortion_k2>
-          <distortion_k3>0.0</distortion_k3>
-          <distortion_t1>0.0</distortion_t1>
-          <distortion_t2>0.0</distortion_t2>
-          <pointCloudCutoff>0.4</pointCloudCutoff>
-        </plugin>
-      </sensor>
-    </gazebo>
-  </xacro:macro>
   <!-- add sensor part -->
-<!-- add sensor camera LEFT part -->
-  <xacro:macro name="sim_3dsensor" params="prefix">
-    <gazebo reference="${prefix}_depth_frame">
-      <sensor type="depth" name="camera">
-        <always_on>true</always_on>
-        <update_rate>20.0</update_rate>
-        <camera>
-          <horizontal_fov>${60.0*pi/180.0}</horizontal_fov>
-          <image>
-            <format>B8G8R8</format>
-            <width>640</width>
-            <height>480</height>
-          </image>  <xacro:macro name="sim_3dsensor" params="prefix">
+  <!-- add sensor camera LEFT part -->
+  <!-- <xacro:macro name="sim_3dsensor" params="prefix">
     <gazebo reference="${prefix}_depth_frame">
       <sensor type="depth" name="camera">
@@ -127,31 +79,5 @@
       </sensor>
     </gazebo>
-  </xacro:macro>
-          <clip>
-            <near>0.10</near>
-            <far>8.0</far>
-          </clip>
-        </camera>
-        <plugin name="${prefix}_camera_controller" filename="libgazebo_ros_openni_kinect.so">
-          <cameraName>${prefix}</cameraName>
-          <alwaysOn>true</alwaysOn>
-          <updateRate>10</updateRate>
-          <imageTopicName>rgb/image_raw</imageTopicName>
-          <depthImageTopicName>depth/image_raw</depthImageTopicName>
-          <pointCloudTopicName>depth/points</pointCloudTopicName>
-          <cameraInfoTopicName>rgb/camera_info</cameraInfoTopicName>
-          <depthImageCameraInfoTopicName>depth/camera_info</depthImageCameraInfoTopicName>
-          <frameName>${prefix}_depth_optical_frame</frameName>
-          <baseline>0.1</baseline>
-          <distortion_k1>0.0</distortion_k1>
-          <distortion_k2>0.0</distortion_k2>
-          <distortion_k3>0.0</distortion_k3>
-          <distortion_t1>0.0</distortion_t1>
-          <distortion_t2>0.0</distortion_t2>
-          <pointCloudCutoff>0.4</pointCloudCutoff>
-        </plugin>
-      </sensor>
-    </gazebo>
-  </xacro:macro>
+  </xacro:macro> -->
   <!-- add sensor part -->
 </robot>

File: tripod_calibration_test/tripod_calib_test_description/urdf/tripod_rgb_rgb.urdf.xacro (robot description, xacro)
@@ -15,5 +15,5 @@
     </xacro:sensor_astra>
     <!-- ADD CHESSBOARD -->
-    <xacro:include filename="$(find tripod_calib_test_description)/models/charuco5X5.urdf.xacro" />
+    <!-- <xacro:include filename="$(find tripod_calib_test_description)/models/charuco5X5.urdf.xacro" /> -->
     <material name="grey">
         <color rgba="0.7 0.7 0.7 1.0" />
