Commit message: rename files to tripod_rgb_rgb

File: tripod_rgb_rgb/tripod_rgb_rgb_description/models/charuco5X5.urdf.xacro (robot description, xacro)
@@ -9,5 +9,5 @@
         <visual>
             <geometry>
-                <mesh filename="package://tripod_calib_test_description/meshes/objects/charuco_5x5.dae" />
+                <mesh filename="package://tripod_rgb_rgb_description/meshes/objects/charuco_5x5.dae" />
                 <!-- <box size="0.3 0.2 0.01" /> -->
             </geometry>

File: tripod_rgb_rgb/tripod_rgb_rgb_description/urdf/astra.urdf.xacro (robot description, xacro)
@@ -1,5 +1,5 @@
 <?xml version="1.0"?>
 <robot name="sensor_astra" xmlns:xacro="http://ros.org/wiki/xacro">
-  <xacro:include filename="$(find tripod_calib_test_description)/urdf/tripod_rgb_rgb.gazebo.xacro" />
+  <xacro:include filename="$(find tripod_rgb_rgb_description)/urdf/tripod_rgb_rgb.gazebo.xacro" />
   <!-- Xacro properties -->
   <xacro:property name="astra_cam_py" value="-0.0125"/>
@@ -18,5 +18,5 @@
         <origin xyz="-0.03 -0.06 0" rpy="${pi} 0 ${pi/2}"/>
         <geometry>
-          <mesh filename="package://tripod_calib_test_description/meshes/sensors/astra2.dae" scale="1 1 1"/>
+          <mesh filename="package://tripod_rgb_rgb_description/meshes/sensors/astra2.dae" scale="1 1 1"/>
         </geometry>
       </visual>

File: tripod_rgb_rgb/tripod_rgb_rgb_description/urdf/tripod_rgb_rgb.urdf.xacro (robot description, xacro)
@@ -3,5 +3,5 @@
     <xacro:property name="M_PI" value="3.1415926535897931" />
     <!-- testing adding a sensor camera -->
-    <xacro:include filename="$(find tripod_calib_test_description)/urdf/astra.urdf.xacro" />
+    <xacro:include filename="$(find tripod_rgb_rgb_description)/urdf/astra.urdf.xacro" />
     <!-- RIGHT CAMERA -->
     <xacro:sensor_astra parent="tripod_right_support" prefix="cameraR">
@@ -15,5 +15,5 @@
     </xacro:sensor_astra>
     <!-- ADD charuco REMOVED FROM HERE TO BE SEEN AS A DIFFERENT OBJECT IN THE SIMULATION -->
-    <!-- <xacro:include filename="$(find tripod_calib_test_description)/models/charuco5X5.urdf.xacro" /> -->
+    <!-- <xacro:include filename="$(find tripod_rgb_rgb_description)/models/charuco5X5.urdf.xacro" /> -->
     <material name="grey">
         <color rgba="0.7 0.7 0.7 1.0" />
@@ -25,5 +25,5 @@
             <origin xyz="0 0 0" rpy="0 0 0" />
             <geometry>
-                <mesh filename="package://tripod_calib_test_description/meshes/tripod/tripod.dae" scale="0.04 0.04 0.04" />
+                <mesh filename="package://tripod_rgb_rgb_description/meshes/tripod/tripod.dae" scale="0.04 0.04 0.04" />
             </geometry>
             <material name="grey" />
@@ -32,5 +32,5 @@
             <origin xyz="0 0 0" rpy="0 0 0" />
             <geometry>
-                <mesh filename="package://tripod_calib_test_description/meshes/tripod/tripod.dae" scale="0.04 0.04 0.04" />
+                <mesh filename="package://tripod_rgb_rgb_description/meshes/tripod/tripod.dae" scale="0.04 0.04 0.04" />
             </geometry>
         </collision>

File: tripod_rgb_rgb_calibration/urdf/initial_estimate.urdf.xacro (robot description, xacro)
@@ -1,261 +1,117 @@
-<?xml version="1.0" ?>
-<robot name="tripod_macro" version="1.0">
-  <joint name="cameraR_joint" type="fixed">
-    <origin xyz="0.0 0.05 0.015" rpy="0.0 -0.0 0.0"/>
-    <parent link="tripod_right_support"/>
-    <child link="cameraR_link"/>
-  </joint>
-  <link name="cameraR_link">
-    <inertial>
-      <origin xyz="0.0 0.0 0.0" rpy="0 0 0"/>
-      <mass value="0.564"/>
-      <inertia ixx="0.003881243" ixy="0.0" ixz="0.0" iyy="0.00049894" iyz="0.0" izz="0.003879257"/>
-    </inertial>
-    <visual>
-      <origin xyz="-0.03 -0.06 0.0" rpy="3.141592653589793 0.0 1.5707963267948966"/>
-      <geometry>
-        <mesh filename="package://tripod_calib_test_description/meshes/sensors/astra2.dae" scale="1.0 1.0 1.0"/>
-      </geometry>
-    </visual>
-    <collision>
-      <origin xyz="-0.01 -0.06 0.0" rpy="0.0 0.0 0.0"/>
-      <geometry>
-        <box size="0.04 0.165 0.03"/>
-      </geometry>
-    </collision>
-  </link>
-  <joint name="cameraR_rgb_joint" type="fixed">
-    <origin xyz="0.0 -0.045 0.0" rpy="0.0 0.0 0.0"/>
-    <parent link="cameraR_link"/>
-    <child link="cameraR_rgb_frame"/>
-  </joint>
-  <link name="cameraR_rgb_frame"/>
-  <joint name="cameraR_rgb_optical_joint" type="fixed">
-    <origin xyz="0.0 0.0 0.0" rpy="-1.5707963267948966 0.0 -1.5707963267948966"/>
-    <parent link="cameraR_rgb_frame"/>
-    <child link="cameraR_rgb_optical_frame"/>
-  </joint>
-  <link name="cameraR_rgb_optical_frame"/>
-  <joint name="cameraR_depth_joint" type="fixed">
-    <origin xyz="0.0 -0.02 0.0" rpy="0.0 0.0 0.0"/>
-    <parent link="cameraR_link"/>
-    <child link="cameraR_depth_frame"/>
-  </joint>
-  <link name="cameraR_depth_frame"/>
-  <joint name="cameraR_depth_optical_joint" type="fixed">
-    <origin xyz="0.0 0.0 0.0" rpy="-1.5707963267948966 0.0 -1.5707963267948966"/>
-    <parent link="cameraR_depth_frame"/>
-    <child link="cameraR_depth_optical_frame"/>
-  </joint>
-  <link name="cameraR_depth_optical_frame"/>
-  <gazebo reference="cameraR_depth_frame">
-    <sensor name="camera" type="depth">
-      <always_on>true</always_on>
-      <update_rate>20.0</update_rate>
-      <camera>
-        <horizontal_fov>1.0471975511965976</horizontal_fov>
-        <image>
-          <format>B8G8R8</format>
-          <width>640</width>
-          <height>480</height>
-        </image>
-        <clip>
-          <near>0.10</near>
-          <far>8.0</far>
-        </clip>
-      </camera>
-      <plugin filename="libgazebo_ros_openni_kinect.so" name="cameraR_camera_controller">
-        <cameraName>cameraR</cameraName>
-        <alwaysOn>true</alwaysOn>
-        <updateRate>10</updateRate>
-        <imageTopicName>rgb/image_raw</imageTopicName>
-        <depthImageTopicName>depth/image_raw</depthImageTopicName>
-        <pointCloudTopicName>depth/points</pointCloudTopicName>
-        <cameraInfoTopicName>rgb/camera_info</cameraInfoTopicName>
-        <depthImageCameraInfoTopicName>depth/camera_info</depthImageCameraInfoTopicName>
-        <frameName>cameraR_depth_optical_frame</frameName>
-        <baseline>0.1</baseline>
-        <distortion_k1>0.0</distortion_k1>
-        <distortion_k2>0.0</distortion_k2>
-        <distortion_k3>0.0</distortion_k3>
-        <distortion_t1>0.0</distortion_t1>
-        <distortion_t2>0.0</distortion_t2>
-        <pointCloudCutoff>0.4</pointCloudCutoff>
-      </plugin>
-    </sensor>
-  </gazebo>
-  <joint name="cameraL_joint" type="fixed">
-    <origin xyz="0.0 0.075 0.015" rpy="0.0 -0.0 0.0"/>
-    <parent link="tripod_left_support"/>
-    <child link="cameraL_link"/>
-  </joint>
-  <link name="cameraL_link">
-    <inertial>
-      <origin xyz="0.0 0.0 0.0" rpy="0 0 0"/>
-      <mass value="0.564"/>
-      <inertia ixx="0.003881243" ixy="0.0" ixz="0.0" iyy="0.00049894" iyz="0.0" izz="0.003879257"/>
-    </inertial>
-    <visual>
-      <origin xyz="-0.03 -0.06 0.0" rpy="3.141592653589793 0.0 1.5707963267948966"/>
-      <geometry>
-        <mesh filename="package://tripod_calib_test_description/meshes/sensors/astra2.dae" scale="1.0 1.0 1.0"/>
-      </geometry>
-    </visual>
-    <collision>
-      <origin xyz="-0.01 -0.06 0.0" rpy="0.0 0.0 0.0"/>
-      <geometry>
-        <box size="0.04 0.165 0.03"/>
-      </geometry>
-    </collision>
-  </link>
-  <joint name="cameraL_rgb_joint" type="fixed">
-    <origin xyz="0.0 -0.045 0.0" rpy="0.0 0.0 0.0"/>
-    <parent link="cameraL_link"/>
-    <child link="cameraL_rgb_frame"/>
-  </joint>
-  <link name="cameraL_rgb_frame"/>
-  <joint name="cameraL_rgb_optical_joint" type="fixed">
-    <origin xyz="0.0 0.0 0.0" rpy="-1.5707963267948966 0.0 -1.5707963267948966"/>
-    <parent link="cameraL_rgb_frame"/>
-    <child link="cameraL_rgb_optical_frame"/>
-  </joint>
-  <link name="cameraL_rgb_optical_frame"/>
-  <joint name="cameraL_depth_joint" type="fixed">
-    <origin xyz="0.0 -0.02 0.0" rpy="0.0 0.0 0.0"/>
-    <parent link="cameraL_link"/>
-    <child link="cameraL_depth_frame"/>
-  </joint>
-  <link name="cameraL_depth_frame"/>
-  <joint name="cameraL_depth_optical_joint" type="fixed">
-    <origin xyz="0.0 0.0 0.0" rpy="-1.5707963267948966 0.0 -1.5707963267948966"/>
-    <parent link="cameraL_depth_frame"/>
-    <child link="cameraL_depth_optical_frame"/>
-  </joint>
-  <link name="cameraL_depth_optical_frame"/>
-  <gazebo reference="cameraL_depth_frame">
-    <sensor name="camera" type="depth">
-      <always_on>true</always_on>
-      <update_rate>20.0</update_rate>
-      <camera>
-        <horizontal_fov>1.0471975511965976</horizontal_fov>
-        <image>
-          <format>B8G8R8</format>
-          <width>640</width>
-          <height>480</height>
-        </image>
-        <clip>
-          <near>0.10</near>
-          <far>8.0</far>
-        </clip>
-      </camera>
-      <plugin filename="libgazebo_ros_openni_kinect.so" name="cameraL_camera_controller">
-        <cameraName>cameraL</cameraName>
-        <alwaysOn>true</alwaysOn>
-        <updateRate>10</updateRate>
-        <imageTopicName>rgb/image_raw</imageTopicName>
-        <depthImageTopicName>depth/image_raw</depthImageTopicName>
-        <pointCloudTopicName>depth/points</pointCloudTopicName>
-        <cameraInfoTopicName>rgb/camera_info</cameraInfoTopicName>
-        <depthImageCameraInfoTopicName>depth/camera_info</depthImageCameraInfoTopicName>
-        <frameName>cameraL_depth_optical_frame</frameName>
-        <baseline>0.1</baseline>
-        <distortion_k1>0.0</distortion_k1>
-        <distortion_k2>0.0</distortion_k2>
-        <distortion_k3>0.0</distortion_k3>
-        <distortion_t1>0.0</distortion_t1>
-        <distortion_t2>0.0</distortion_t2>
-        <pointCloudCutoff>0.4</pointCloudCutoff>
-      </plugin>
-    </sensor>
-  </gazebo>
-  <material name="grey">
-    <color rgba="0.7 0.7 0.7 1.0"/>
-  </material>
-  <link name="world"/>
-  <link name="tripod">
-    <inertial>
-      <origin xyz="0.0 0.0 0.0" rpy="0.0 0.0 0.0"/>
-      <mass value="1.0"/>
-      <inertia ixx="1.0" ixy="0.0" ixz="0.0" iyy="1.0" iyz="0.0" izz="1.0"/>
-    </inertial>
-    <visual>
-      <origin xyz="0.0 0.0 0.0" rpy="0.0 0.0 0.0"/>
-      <geometry>
-        <mesh filename="package://tripod_calib_test_description/meshes/tripod/tripod.dae" scale="0.04 0.04 0.04"/>
-      </geometry>
-      <material name="grey"/>
-    </visual>
-    <collision name="tripod_collision">
-      <origin xyz="0.0 0.0 0.0" rpy="0.0 0.0 0.0"/>
-      <geometry>
-        <mesh filename="package://tripod_calib_test_description/meshes/tripod/tripod.dae" scale="0.04 0.04 0.04"/>
-      </geometry>
-    </collision>
-  </link>
-  <gazebo reference="tripod">
-    <material>Gazebo/Grey</material>
-    <mu1>50.0</mu1>
-    <mu2>50.0</mu2>
-    <kp>1000000.0</kp>
-    <kd>1.0</kd>
-    <selfCollide>false</selfCollide>
-  </gazebo>
-  <joint name="world_to_tripod" type="fixed">
-    <origin xyz="0.0 0.0 0.0" rpy="0.0 0.0 0.0"/>
-    <parent link="world"/>
-    <child link="tripod"/>
-  </joint>
-  <gazebo reference="tripod">
-    <material>Gazebo/Grey</material>
-    <mu1>50.0</mu1>
-    <mu2>50.0</mu2>
-    <kp>1000000.0</kp>
-    <kd>1.0</kd>
-    <selfCollide>false</selfCollide>
-  </gazebo>
-  <link name="tripod_plate">
-    <inertial>
-      <origin xyz="0.0 0.0 0.0" rpy="0.0 0.0 0.0"/>
-      <mass value="1.0"/>
-      <inertia ixx="1.0" ixy="0.0" ixz="0.0" iyy="1.0" iyz="0.0" izz="1.0"/>
-    </inertial>
-    <visual>
-      <origin xyz="0.0 0.0 0.0" rpy="0.0 0.0 0.0"/>
-      <geometry>
-        <box size="0.04 0.4 0.015"/>
-      </geometry>
-      <material name="grey"/>
-    </visual>
-    <collision name="tripod_collision">
-      <origin xyz="0.0 0.0 0.0" rpy="0.0 0.0 0.0"/>
-      <geometry>
-        <box size="0.04 0.15 0.015"/>
-      </geometry>
-    </collision>
-  </link>
-  <gazebo reference="tripod">
-    <material>Gazebo/Grey</material>
-    <mu1>50.0</mu1>
-    <mu2>50.0</mu2>
-    <kp>1000000.0</kp>
-    <kd>1.0</kd>
-    <selfCollide>false</selfCollide>
-  </gazebo>
-  <joint name="tripod_to_tripod_plate" type="fixed">
-    <origin xyz="0.01 0.03 1.33" rpy="0.0 0.3141592653589793 0.0"/>
-    <parent link="tripod"/>
-    <child link="tripod_plate"/>
-  </joint>
-  <link name="tripod_left_support"/>
-  <joint name="tripod_plate_to_tripod_left_support" type="fixed">
-    <origin xyz="0.0 0.18 0.0075" rpy="0.0 0.0 0.0"/>
-    <parent link="tripod_plate"/>
-    <child link="tripod_left_support"/>
-  </joint>
-  <link name="tripod_right_support"/>
-  <joint name="tripod_plate_to_tripod_right_support" type="fixed">
-    <origin xyz="0.0 -0.18 0.0075" rpy="0.0 0.0 0.0"/>
-    <parent link="tripod_plate"/>
-    <child link="tripod_right_support"/>
-  </joint>
+<?xml version="1.0"?>
+<robot name="tripod_macro" xmlns:xacro="http://ros.org/wiki/xacro">
+    <xacro:property name="M_PI" value="3.1415926535897931" />
+    <!-- testing adding a sensor camera -->
+    <xacro:include filename="$(find tripod_rgb_rgb_description)/urdf/astra.urdf.xacro" />
+    <!-- RIGHT CAMERA -->
+    <xacro:sensor_astra parent="tripod_right_support" prefix="cameraR">
+        <origin xyz="0 0.05 0.015"
+            rpy="0 0 0" />
+    </xacro:sensor_astra>
+    <!-- LEFT CAMERA -->
+    <xacro:sensor_astra parent="tripod_left_support" prefix="cameraL">
+        <origin xyz="0 0.075 0.015"
+            rpy="0 0 0" />
+    </xacro:sensor_astra>
+    <!-- ADD charuco REMOVED FROM HERE TO BE SEEN AS A DIFFERENT OBJECT IN THE SIMULATION -->
+    <!-- <xacro:include filename="$(find tripod_rgb_rgb_description)/models/charuco5X5.urdf.xacro" /> -->
+    <material name="grey">
+        <color rgba="0.7 0.7 0.7 1.0" />
+    </material>
+    <link name="world" />
+    <!-- Tripod link-->
+    <link name="tripod">
+        <visual>
+            <origin xyz="0 0 0" rpy="0 0 0" />
+            <geometry>
+                <mesh filename="package://tripod_rgb_rgb_description/meshes/tripod/tripod.dae" scale="0.04 0.04 0.04" />
+            </geometry>
+            <material name="grey" />
+        </visual>
+        <collision name="tripod_collision">
+            <origin xyz="0 0 0" rpy="0 0 0" />
+            <geometry>
+                <mesh filename="package://tripod_rgb_rgb_description/meshes/tripod/tripod.dae" scale="0.04 0.04 0.04" />
+            </geometry>
+        </collision>
+        <inertial>
+            <mass value="1.0" />
+            <origin xyz="0 0 0" rpy="0 0 0" />
+            <inertia ixx="1" ixy="0" ixz="0" iyy="1" iyz="0" izz="1" />
+        </inertial>
+    </link>
+    <gazebo reference="tripod">
+        <material>Gazebo/Grey</material>
+        <mu1>50.0</mu1>
+        <mu2>50.0</mu2>
+        <kp>1000000.0</kp>
+        <kd>1.0</kd>
+        <selfCollide>false</selfCollide>
+    </gazebo>
+    <!-- parent to tripod -->
+    <joint name="world_to_tripod" type="fixed">
+        <parent link="world" />
+        <child link="tripod" />
+        <!-- <xacro:insert_block name="origin" /> -->
+        <origin xyz="0 0 0" rpy="0 0 0" />
+    </joint>
+    <gazebo reference="tripod">
+        <material>Gazebo/Grey</material>
+        <mu1>50.0</mu1>
+        <mu2>50.0</mu2>
+        <kp>1000000.0</kp>
+        <kd>1.0</kd>
+        <selfCollide>false</selfCollide>
+    </gazebo>
+    <link name="tripod_plate">
+        <visual>
+            <origin xyz="0 0 0" rpy="0 0 0" />
+            <geometry>
+                <box size="0.04 0.4 0.015" />
+            </geometry>
+            <material name="grey" />
+        </visual>
+        <collision name="tripod_collision">
+            <origin xyz="0 0 0" rpy="0 0 0" />
+            <geometry>
+                <box size="0.04 0.15 0.015" />
+            </geometry>
+        </collision>
+        <inertial>
+            <mass value="1.0" />
+            <origin xyz="0 0 0" rpy="0 0 0" />
+            <inertia ixx="1" ixy="0" ixz="0" iyy="1" iyz="0" izz="1" />
+        </inertial>
+    </link>
+    <gazebo reference="tripod">
+        <material>Gazebo/Grey</material>
+        <mu1>50.0</mu1>
+        <mu2>50.0</mu2>
+        <kp>1000000.0</kp>
+        <kd>1.0</kd>
+        <selfCollide>false</selfCollide>
+    </gazebo>
+    <!-- tripod to tripod plate-->
+    <joint name="tripod_to_tripod_plate" type="fixed">
+        <parent link="tripod" />
+        <child link="tripod_plate" />
+        <origin xyz=".01 .03 1.33" rpy="0 ${M_PI/10} 0" />
+    </joint>
+    <!-- Tripod left support-->
+    <link name="tripod_left_support" />
+    <!-- tripod plate to tripod left support -->
+    <joint name="tripod_plate_to_tripod_left_support" type="fixed">
+        <parent link="tripod_plate" />
+        <child link="tripod_left_support" />
+        <origin xyz="0 0.18 0.0075" rpy="0 0 0" />
+    </joint>
+    <!-- Tripod right support-->
+    <link name="tripod_right_support" />
+    <!-- tripod plate to tripod right support -->
+    <joint name="tripod_plate_to_tripod_right_support" type="fixed">
+        <parent link="tripod_plate" />
+        <child link="tripod_right_support" />
+        <origin xyz="0 -0.18 0.0075" rpy="0 0 0" />
+    </joint>
+    <!-- </xacro:macro> -->
 </robot>
