Commit message: t2rgb ATOM calibration

File: t2rgb_description/urdf/astra.urdf.xacro (robot description, xacro)
@@ -3,28 +3,28 @@
   <xacro:include filename="$(find t2rgb_description)/urdf/t2rgb.gazebo.xacro" />
   <!-- Xacro properties -->
-  <xacro:property name="astra_cam_py" value="-0.0125"/>
+  <xacro:property name="astra_cam_py" value="-0.0125" />
   <xacro:property name="astra_depth_rel_rgb_py" value="0.0250" />
-  <xacro:property name="astra_cam_rel_rgb_py"   value="-0.0125" />
-  <xacro:property name="astra_dae_display_scale"   value="0.1" />
+  <xacro:property name="astra_cam_rel_rgb_py" value="-0.0125" />
+  <xacro:property name="astra_dae_display_scale" value="0.1" />
   <!-- Parameterised in part by the values in turtlebot_properties.urdf.xacro -->
   <xacro:macro name="sensor_astra" params="parent prefix *origin">
     <joint name="${prefix}_joint" type="fixed">
       <xacro:insert_block name="origin" />
-      <parent link="${parent}"/>
-      <child link="${prefix}_link"/>
+      <parent link="${parent}" />
+      <child link="${prefix}_link" />
     </joint>
     <link name="${prefix}_link">
-      <visual>
+      <!-- <visual>
         <origin xyz="-0.03 -0.06 0" rpy="${pi} 0 ${pi/2}"/>
         <geometry>
           <mesh filename="package://t2rgb_description/meshes/sensors/astra2.dae" scale="1 1 1"/>
         </geometry>
-      </visual>
+      </visual> -->
       <collision>
         <!-- <origin xyz="0.0 0.0 0.0" rpy="0 0 0" /> -->
-        <origin xyz="-0.01 -0.06 0" rpy="0 0 0"/>
+        <origin xyz="-0.01 -0.06 0" rpy="0 0 0" />
         <geometry>
-        <box size="0.0400 0.1650 0.0300"/>
-      </geometry>
+          <box size="0.0400 0.1650 0.0300" />
+        </geometry>
       </collision>
       <inertial>
@@ -32,14 +32,18 @@
         <origin xyz="0 0 0" />
         <inertia ixx="0.003881243" ixy="0.0" ixz="0.0"
-                 iyy="0.000498940" iyz="0.0"
-                 izz="0.003879257" />
+          iyy="0.000498940" iyz="0.0"
+          izz="0.003879257" />
       </inertial>
     </link>
+    <!-- add to improve set initial pose on atom -->
+    <gazebo reference="${prefix}_link">
+      <selfCollide>false</selfCollide>
+    </gazebo>
     <joint name="${prefix}_rgb_joint" type="fixed">
       <origin xyz="0 -0.045 0" rpy="0 0 0" />
-      <parent link="${prefix}_link"/>
+      <parent link="${prefix}_link" />
       <child link="${prefix}_rgb_frame" />
     </joint>
-    <link name="${prefix}_rgb_frame"/>
+    <link name="${prefix}_rgb_frame" />
     <joint name="${prefix}_rgb_optical_joint" type="fixed">
       <origin xyz="0 0 0" rpy="${-pi/2} 0 ${-pi/2}" />
@@ -47,17 +51,34 @@
       <child link="${prefix}_rgb_optical_frame" />
     </joint>
-    <link name="${prefix}_rgb_optical_frame"/>
+    <!-- add to improve set initial pose on atom -->
+    <link name="${prefix}_rgb_optical_frame">
+      <visual>
+        <origin xyz="0.0 0.0 -0.03" rpy="${pi/2} 0 0" />
+        <geometry>
+          <mesh filename="package://t2rgb_description/meshes/sensors/astra2.dae" scale="1 1 1" />
+        </geometry>
+      </visual>
+    </link>
     <joint name="${prefix}_depth_joint" type="fixed">
-        <origin xyz="0 -0.02 0" rpy="0 0 0" />
-        <parent link="${prefix}_link" />
-        <child link="${prefix}_depth_frame" />
+      <origin xyz="0 -0.02 0" rpy="0 0 0" />
+      <parent link="${prefix}_link" />
+      <child link="${prefix}_depth_frame" />
     </joint>
-    <link name="${prefix}_depth_frame"/>
+    <link name="${prefix}_depth_frame" />
     <joint name="${prefix}_depth_optical_joint" type="fixed">
-        <origin xyz="0 0 0" rpy="${-pi/2} 0 ${-pi/2}" />
-        <parent link="${prefix}_depth_frame" />
-        <child link="${prefix}_depth_optical_frame" />
+      <origin xyz="0 0 0" rpy="${-pi/2} 0 ${-pi/2}" />
+      <parent link="${prefix}_depth_frame" />
+      <child link="${prefix}_depth_optical_frame" />
     </joint>
-    <link name="${prefix}_depth_optical_frame"/>
+    <!-- add to improve set initial pose on atom -->
+    <link name="${prefix}_depth_optical_frame">
+      <!-- <visual>
+        <origin xyz="0.0 0.0 0.0" rpy="0 0 0" />
+        <geometry> -->
+          <!-- Use a slightly smaller scale than 1, so that when both models overlap its the rgb that appears.-->
+          <!-- <mesh filename="package://t2rgb_description/meshes/sensors/astra2.dae" scale="0.98 0.98 0.98" />
+        </geometry>
+      </visual> -->
+    </link>
     <xacro:sim_3dsensor prefix="${prefix}" />
   </xacro:macro>

File: t2rgb_description/urdf/optimized.urdf.xacro (robot description, xacro)
@@ -23,5 +23,5 @@
   </gazebo>
   <joint name="camera_right_rgb_joint" type="fixed">
-    <origin xyz="0.0 -0.045 0.0" rpy="0.0 -0.0 0.0"/>
+    <origin xyz="0.0005209253551980347 -0.03617339647319985 -0.011479420546483453" rpy="0.01843166991852172 -0.0034089482428418263 0.004603148305513264"/>
     <parent link="camera_right_link"/>
     <child link="camera_right_rgb_frame"/>
@@ -111,5 +111,5 @@
   </gazebo>
   <joint name="camera_left_rgb_joint" type="fixed">
-    <origin xyz="0.0 -0.045 0.0" rpy="0.0 -0.0 0.0"/>
+    <origin xyz="-0.0019452346314990437 -0.03864037374945174 -0.004458487237583798" rpy="0.018296669584651013 -0.003460658961089324 0.006472138607952493"/>
     <parent link="camera_left_link"/>
     <child link="camera_left_rgb_frame"/>

File: t2rgb_description/urdf/optimized/optimized_2022_11_19-02_08_33_PM.urdf.xacro (robot description, xacro)
@@ -1,19 +1,19 @@
-<?xml version="1.0" ?>
+<?xml version="1.0"?>
 <robot name="tripod_macro" version="1.0">
   <joint name="camera_right_joint" type="fixed">
-    <origin xyz="0.0 0.05 0.015" rpy="0.0 0.0 0.0"/>
-    <parent link="tripod_right_support"/>
-    <child link="camera_right_link"/>
+    <origin xyz="0.0 0.05 0.015" rpy="0.0 0.0 0.0" />
+    <parent link="tripod_right_support" />
+    <child link="camera_right_link" />
   </joint>
   <link name="camera_right_link">
     <inertial>
-      <origin xyz="0.0 0.0 0.0" rpy="0 0 0"/>
-      <mass value="0.564"/>
-      <inertia ixx="0.003881243" ixy="0.0" ixz="0.0" iyy="0.00049894" iyz="0.0" izz="0.003879257"/>
+      <origin xyz="0.0 0.0 0.0" rpy="0 0 0" />
+      <mass value="0.564" />
+      <inertia ixx="0.003881243" ixy="0.0" ixz="0.0" iyy="0.00049894" iyz="0.0" izz="0.003879257" />
     </inertial>
     <collision>
-      <origin xyz="-0.01 -0.06 0.0" rpy="0.0 0.0 0.0"/>
-      <geometry>
-        <box size="0.04 0.165 0.03"/>
+      <origin xyz="-0.01 -0.06 0.0" rpy="0.0 0.0 0.0" />
+      <geometry>
+        <box size="0.04 0.165 0.03" />
       </geometry>
     </collision>
@@ -23,34 +23,34 @@
   </gazebo>
   <joint name="camera_right_rgb_joint" type="fixed">
-    <origin xyz="0.0 -0.045 0.0" rpy="0.0 -0.0 0.0"/>
-    <parent link="camera_right_link"/>
-    <child link="camera_right_rgb_frame"/>
-  </joint>
-  <link name="camera_right_rgb_frame"/>
+    <origin xyz="0.0005209253551980347 -0.03617339647319985 -0.011479420546483453" rpy="0.01843166991852172 -0.0034089482428418263 0.004603148305513264" />
+    <parent link="camera_right_link" />
+    <child link="camera_right_rgb_frame" />
+  </joint>
+  <link name="camera_right_rgb_frame" />
   <joint name="camera_right_rgb_optical_joint" type="fixed">
-    <origin xyz="0.0 0.0 0.0" rpy="-1.5707963267948966 0.0 -1.5707963267948966"/>
-    <parent link="camera_right_rgb_frame"/>
-    <child link="camera_right_rgb_optical_frame"/>
+    <origin xyz="0.0 0.0 0.0" rpy="-1.5707963267948966 0.0 -1.5707963267948966" />
+    <parent link="camera_right_rgb_frame" />
+    <child link="camera_right_rgb_optical_frame" />
   </joint>
   <link name="camera_right_rgb_optical_frame">
     <visual>
-      <origin xyz="0.0 0.0 -0.03" rpy="1.5707963267948966 0.0 0.0"/>
-      <geometry>
-        <mesh filename="package://t2rgb_description/meshes/sensors/astra2.dae" scale="1.0 1.0 1.0"/>
+      <origin xyz="0.0 0.0 -0.03" rpy="1.5707963267948966 0.0 0.0" />
+      <geometry>
+        <mesh filename="package://t2rgb_description/meshes/sensors/astra2.dae" scale="1.0 1.0 1.0" />
       </geometry>
     </visual>
   </link>
   <joint name="camera_right_depth_joint" type="fixed">
-    <origin xyz="0.0 -0.02 0.0" rpy="0.0 0.0 0.0"/>
-    <parent link="camera_right_link"/>
-    <child link="camera_right_depth_frame"/>
-  </joint>
-  <link name="camera_right_depth_frame"/>
+    <origin xyz="0.0 -0.02 0.0" rpy="0.0 0.0 0.0" />
+    <parent link="camera_right_link" />
+    <child link="camera_right_depth_frame" />
+  </joint>
+  <link name="camera_right_depth_frame" />
   <joint name="camera_right_depth_optical_joint" type="fixed">
-    <origin xyz="0.0 0.0 0.0" rpy="-1.5707963267948966 0.0 -1.5707963267948966"/>
-    <parent link="camera_right_depth_frame"/>
-    <child link="camera_right_depth_optical_frame"/>
-  </joint>
-  <link name="camera_right_depth_optical_frame"/>
+    <origin xyz="0.0 0.0 0.0" rpy="-1.5707963267948966 0.0 -1.5707963267948966" />
+    <parent link="camera_right_depth_frame" />
+    <child link="camera_right_depth_optical_frame" />
+  </joint>
+  <link name="camera_right_depth_optical_frame" />
   <gazebo reference="camera_right_depth_frame">
     <sensor name="camera" type="depth">
@@ -90,18 +90,18 @@
   </gazebo>
   <joint name="camera_left_joint" type="fixed">
-    <origin xyz="0.0 0.075 0.015" rpy="0.0 0.0 0.0"/>
-    <parent link="tripod_left_support"/>
-    <child link="camera_left_link"/>
+    <origin xyz="0.0 0.075 0.015" rpy="0.0 0.0 0.0" />
+    <parent link="tripod_left_support" />
+    <child link="camera_left_link" />
   </joint>
   <link name="camera_left_link">
     <inertial>
-      <origin xyz="0.0 0.0 0.0" rpy="0 0 0"/>
-      <mass value="0.564"/>
-      <inertia ixx="0.003881243" ixy="0.0" ixz="0.0" iyy="0.00049894" iyz="0.0" izz="0.003879257"/>
+      <origin xyz="0.0 0.0 0.0" rpy="0 0 0" />
+      <mass value="0.564" />
+      <inertia ixx="0.003881243" ixy="0.0" ixz="0.0" iyy="0.00049894" iyz="0.0" izz="0.003879257" />
     </inertial>
     <collision>
-      <origin xyz="-0.01 -0.06 0.0" rpy="0.0 0.0 0.0"/>
-      <geometry>
-        <box size="0.04 0.165 0.03"/>
+      <origin xyz="-0.01 -0.06 0.0" rpy="0.0 0.0 0.0" />
+      <geometry>
+        <box size="0.04 0.165 0.03" />
       </geometry>
     </collision>
@@ -111,34 +111,34 @@
   </gazebo>
   <joint name="camera_left_rgb_joint" type="fixed">
-    <origin xyz="0.0 -0.045 0.0" rpy="0.0 -0.0 0.0"/>
-    <parent link="camera_left_link"/>
-    <child link="camera_left_rgb_frame"/>
-  </joint>
-  <link name="camera_left_rgb_frame"/>
+    <origin xyz="-0.0019452346314990437 -0.03864037374945174 -0.004458487237583798" rpy="0.018296669584651013 -0.003460658961089324 0.006472138607952493" />
+    <parent link="camera_left_link" />
+    <child link="camera_left_rgb_frame" />
+  </joint>
+  <link name="camera_left_rgb_frame" />
   <joint name="camera_left_rgb_optical_joint" type="fixed">
-    <origin xyz="0.0 0.0 0.0" rpy="-1.5707963267948966 0.0 -1.5707963267948966"/>
-    <parent link="camera_left_rgb_frame"/>
-    <child link="camera_left_rgb_optical_frame"/>
+    <origin xyz="0.0 0.0 0.0" rpy="-1.5707963267948966 0.0 -1.5707963267948966" />
+    <parent link="camera_left_rgb_frame" />
+    <child link="camera_left_rgb_optical_frame" />
   </joint>
   <link name="camera_left_rgb_optical_frame">
     <visual>
-      <origin xyz="0.0 0.0 -0.03" rpy="1.5707963267948966 0.0 0.0"/>
-      <geometry>
-        <mesh filename="package://t2rgb_description/meshes/sensors/astra2.dae" scale="1.0 1.0 1.0"/>
+      <origin xyz="0.0 0.0 -0.03" rpy="1.5707963267948966 0.0 0.0" />
+      <geometry>
+        <mesh filename="package://t2rgb_description/meshes/sensors/astra2.dae" scale="1.0 1.0 1.0" />
       </geometry>
     </visual>
   </link>
   <joint name="camera_left_depth_joint" type="fixed">
-    <origin xyz="0.0 -0.02 0.0" rpy="0.0 0.0 0.0"/>
-    <parent link="camera_left_link"/>
-    <child link="camera_left_depth_frame"/>
-  </joint>
-  <link name="camera_left_depth_frame"/>
+    <origin xyz="0.0 -0.02 0.0" rpy="0.0 0.0 0.0" />
+    <parent link="camera_left_link" />
+    <child link="camera_left_depth_frame" />
+  </joint>
+  <link name="camera_left_depth_frame" />
   <joint name="camera_left_depth_optical_joint" type="fixed">
-    <origin xyz="0.0 0.0 0.0" rpy="-1.5707963267948966 0.0 -1.5707963267948966"/>
-    <parent link="camera_left_depth_frame"/>
-    <child link="camera_left_depth_optical_frame"/>
-  </joint>
-  <link name="camera_left_depth_optical_frame"/>
+    <origin xyz="0.0 0.0 0.0" rpy="-1.5707963267948966 0.0 -1.5707963267948966" />
+    <parent link="camera_left_depth_frame" />
+    <child link="camera_left_depth_optical_frame" />
+  </joint>
+  <link name="camera_left_depth_optical_frame" />
   <gazebo reference="camera_left_depth_frame">
     <sensor name="camera" type="depth">
@@ -178,24 +178,24 @@
   </gazebo>
   <material name="grey">
-    <color rgba="0.7 0.7 0.7 1.0"/>
+    <color rgba="0.7 0.7 0.7 1.0" />
   </material>
-  <link name="world"/>
+  <link name="world" />
   <link name="tripod">
     <inertial>
-      <origin xyz="0.0 0.0 0.0" rpy="0.0 0.0 0.0"/>
-      <mass value="1.0"/>
-      <inertia ixx="1.0" ixy="0.0" ixz="0.0" iyy="1.0" iyz="0.0" izz="1.0"/>
-    </inertial>
-    <visual>
-      <origin xyz="0.0 0.0 0.0" rpy="0.0 0.0 0.0"/>
-      <geometry>
-        <mesh filename="package://t2rgb_description/meshes/tripod/tripod.dae" scale="0.04 0.04 0.04"/>
-      </geometry>
-      <material name="grey"/>
+      <origin xyz="0.0 0.0 0.0" rpy="0.0 0.0 0.0" />
+      <mass value="1.0" />
+      <inertia ixx="1.0" ixy="0.0" ixz="0.0" iyy="1.0" iyz="0.0" izz="1.0" />
+    </inertial>
+    <visual>
+      <origin xyz="0.0 0.0 0.0" rpy="0.0 0.0 0.0" />
+      <geometry>
+        <mesh filename="package://t2rgb_description/meshes/tripod/tripod.dae" scale="0.04 0.04 0.04" />
+      </geometry>
+      <material name="grey" />
     </visual>
     <collision name="tripod_collision">
-      <origin xyz="0.0 0.0 0.0" rpy="0.0 0.0 0.0"/>
-      <geometry>
-        <mesh filename="package://t2rgb_description/meshes/tripod/tripod.dae" scale="0.04 0.04 0.04"/>
+      <origin xyz="0.0 0.0 0.0" rpy="0.0 0.0 0.0" />
+      <geometry>
+        <mesh filename="package://t2rgb_description/meshes/tripod/tripod.dae" scale="0.04 0.04 0.04" />
       </geometry>
     </collision>
@@ -210,7 +210,7 @@
   </gazebo>
   <joint name="world_to_tripod" type="fixed">
-    <origin xyz="0.0 0.0 0.0" rpy="0.0 0.0 0.0"/>
-    <parent link="world"/>
-    <child link="tripod"/>
+    <origin xyz="0.0 0.0 0.0" rpy="0.0 0.0 0.0" />
+    <parent link="world" />
+    <child link="tripod" />
   </joint>
   <gazebo reference="tripod">
@@ -224,19 +224,19 @@
   <link name="tripod_plate">
     <inertial>
-      <origin xyz="0.0 0.0 0.0" rpy="0.0 0.0 0.0"/>
-      <mass value="1.0"/>
-      <inertia ixx="1.0" ixy="0.0" ixz="0.0" iyy="1.0" iyz="0.0" izz="1.0"/>
-    </inertial>
-    <visual>
-      <origin xyz="0.0 0.0 0.0" rpy="0.0 0.0 0.0"/>
-      <geometry>
-        <box size="0.04 0.4 0.015"/>
-      </geometry>
-      <material name="grey"/>
+      <origin xyz="0.0 0.0 0.0" rpy="0.0 0.0 0.0" />
+      <mass value="1.0" />
+      <inertia ixx="1.0" ixy="0.0" ixz="0.0" iyy="1.0" iyz="0.0" izz="1.0" />
+    </inertial>
+    <visual>
+      <origin xyz="0.0 0.0 0.0" rpy="0.0 0.0 0.0" />
+      <geometry>
+        <box size="0.04 0.4 0.015" />
+      </geometry>
+      <material name="grey" />
     </visual>
     <collision name="tripod_collision">
-      <origin xyz="0.0 0.0 0.0" rpy="0.0 0.0 0.0"/>
-      <geometry>
-        <box size="0.04 0.15 0.015"/>
+      <origin xyz="0.0 0.0 0.0" rpy="0.0 0.0 0.0" />
+      <geometry>
+        <box size="0.04 0.15 0.015" />
       </geometry>
     </collision>
@@ -251,19 +251,19 @@
   </gazebo>
   <joint name="tripod_to_tripod_plate" type="fixed">
-    <origin xyz="0.01 0.03 1.33" rpy="0.0 0.314 0.0"/>
-    <parent link="tripod"/>
-    <child link="tripod_plate"/>
-  </joint>
-  <link name="tripod_left_support"/>
+    <origin xyz="0.01 0.03 1.33" rpy="0.0 0.314 0.0" />
+    <parent link="tripod" />
+    <child link="tripod_plate" />
+  </joint>
+  <link name="tripod_left_support" />
   <joint name="tripod_plate_to_tripod_left_support" type="fixed">
-    <origin xyz="0.0 0.18 0.0075" rpy="0.0 0.0 0.0"/>
-    <parent link="tripod_plate"/>
-    <child link="tripod_left_support"/>
-  </joint>
-  <link name="tripod_right_support"/>
+    <origin xyz="0.0 0.18 0.0075" rpy="0.0 0.0 0.0" />
+    <parent link="tripod_plate" />
+    <child link="tripod_left_support" />
+  </joint>
+  <link name="tripod_right_support" />
   <joint name="tripod_plate_to_tripod_right_support" type="fixed">
-    <origin xyz="0.0 -0.18 0.0075" rpy="0.0 0.0 0.0"/>
-    <parent link="tripod_plate"/>
-    <child link="tripod_right_support"/>
+    <origin xyz="0.0 -0.18 0.0075" rpy="0.0 0.0 0.0" />
+    <parent link="tripod_plate" />
+    <child link="tripod_right_support" />
   </joint>
 </robot>

File: t2rgb_description/urdf/t2rgb.gazebo.xacro (robot description, xacro)
@@ -41,43 +41,3 @@
   </xacro:macro>
   <!-- add sensor part -->
-  <!-- add sensor camera LEFT part -->
-  <!-- <xacro:macro name="sim_3dsensor" params="prefix">
-    <gazebo reference="${prefix}_depth_frame">
-      <sensor type="depth" name="camera">
-        <always_on>true</always_on>
-        <update_rate>20.0</update_rate>
-        <camera>
-          <horizontal_fov>${60.0*pi/180.0}</horizontal_fov>
-          <image>
-            <format>B8G8R8</format>
-            <width>640</width>
-            <height>480</height>
-          </image>
-          <clip>
-            <near>0.10</near>
-            <far>8.0</far>
-          </clip>
-        </camera>
-        <plugin name="${prefix}_camera_controller" filename="libgazebo_ros_openni_kinect.so">
-          <cameraName>${prefix}</cameraName>
-          <alwaysOn>true</alwaysOn>
-          <updateRate>10</updateRate>
-          <imageTopicName>rgb/image_raw</imageTopicName>
-          <depthImageTopicName>depth/image_raw</depthImageTopicName>
-          <pointCloudTopicName>depth/points</pointCloudTopicName>
-          <cameraInfoTopicName>rgb/camera_info</cameraInfoTopicName>
-          <depthImageCameraInfoTopicName>depth/camera_info</depthImageCameraInfoTopicName>
-          <frameName>${prefix}_depth_optical_frame</frameName>
-          <baseline>0.1</baseline>
-          <distortion_k1>0.0</distortion_k1>
-          <distortion_k2>0.0</distortion_k2>
-          <distortion_k3>0.0</distortion_k3>
-          <distortion_t1>0.0</distortion_t1>
-          <distortion_t2>0.0</distortion_t2>
-          <pointCloudCutoff>0.4</pointCloudCutoff>
-        </plugin>
-      </sensor>
-    </gazebo>
-  </xacro:macro> -->
-  <!-- add sensor part -->
 </robot>
